File: main-board-2/electric/scheme/$main-board-2.sch (KiCad schematic (older format))
At the start: 122 parts, among them K1 power-switch, K2 usb-power-switch, P1 batt, P10 rst, P11 screw-1, P13 screw-2, P14 gpio-big, P15 gpio-small, P16 moto-1, P17 moto-2, P3 trigger-btn, P4 CONN_3X2, P7 bootloader, P8 cross board conn, P9 rst, Q1 IRLML2244, Q10 IRLML2244, Q11 sot223, Q12 bc857, Q13 irlml2244, Q2 BC847, Q3 IRLML2244, Q4 IRLML2244, Q5 BC847, Q6 BC847, Q7 BC847, Q8 BC847, Q9 IRLML2244, U5 LM293, U6 L298, U7 MINI-USB-B, X1 8MHz

Commit message: Places zones and made thermal take zones under regulators.
Parts:
- gave numbers to parts that had none: 4
Changed lines of the file:
@@
 Short to gnd should be \ndone using electrolytic \ncapacitor hole.
 $Comp
-L MY_LM317T U?
+L MY_LM317T U2
 U 1 1 52A983AC
 P 3000 1650
-F 0 "U?" H 2800 1850 40  0000 C CNN
+F 0 "U2" H 2800 1850 40  0000 C CNN
 F 1 "MY_LM317T" H 3000 1850 40  0000 L CNN
 F 2 "TO-220" H 3000 1750 30  0000 C CIN
@@
 $EndComp
 $Comp
-L MY_LM317EMP U?
+L MY_LM317EMP U1
 U 1 1 52A983BB
 P 2500 1250
-F 0 "U?" H 2300 1450 40  0000 C CNN
+F 0 "U1" H 2300 1450 40  0000 C CNN
 F 1 "MY_LM317EMP" H 2500 1450 40  0000 L CNN
 F 2 "SOT-223" H 2500 1350 30  0000 C CIN
@@
 Connection ~ 3500 1600
 $Comp
-L MY_LM317EMP U?
+L MY_LM317EMP U3
 U 1 1 52A98839
 P 3300 4000
-F 0 "U?" H 3100 4200 40  0000 C CNN
+F 0 "U3" H 3100 4200 40  0000 C CNN
 F 1 "MY_LM317EMP" H 3300 4200 40  0000 L CNN
 F 2 "SOT-223" H 3300 4100 30  0000 C CIN
@@
 Connection ~ 3800 3950
 $Comp
-L MY_LM317T U?
+L MY_LM317T U4
 U 1 1 52A98A72
 P 3800 4400
-F 0 "U?" H 3600 4600 40  0000 C CNN
+F 0 "U4" H 3600 4600 40  0000 C CNN
 F 1 "MY_LM317T" H 3800 4600 40  0000 L CNN
 F 2 "TO-220" H 3800 4500 30  0000 C CIN
