File: addon-gpio/electric/scheme/addon-gpio.sch (KiCad schematic (older format))
At the start: 69 parts, among them K1 swd, K10 CONN_3, K11 CONN_3, K12 CONN_3, K13 CONN_3, K14 CONN_3, K15 CONN_3, K16 CONN_3, K17 CONN_3, K18 CONN_3, K19 CONN_3, K2 CONN_3, K20 CONN_3, K21 CONN_3, K22 CONN_3, K23 CONN_3, K24 CONN_3, K25 CONN_3, K26 CONN_3, K27 CONN_3, K28 CONN_3, K29 CONN_3, K3 CONN_3, K30 CONN_3, K31 CONN_3, K32 CONN_3, K4 CONN_3, K5 CONN_3, K6 CONN_3, K7 CONN_3, K8 CONN_3, K9 CONN_3, P1 TST, P2 cross board conn, P3 cross board conn, P4 TST, P5 boot-sel, P6 pwr-ext, P7 rst-2, P8 rst-1, Q1 bc847, Q2 sot223, Q3 IRLML2244, Q4 sot223, Q5 IRLML2244, X1 8MHz

Commit message: Routing...
Parts:
- added K33: CONN_3, symbol CONN_3
Connections:
- net labels added: pin_28
- wire segments 319 -> 323
Other:
- moved on the sheet: K10, K11, K12, K18, K19, K5, K6, K7, K8, K9
Changed lines of the file:
@@
 Sheet 1 1
 Title ""
-Date "21 dec 2013"
+Date "22 dec 2013"
 Rev ""
 Comp ""
@@
 Text Notes 17600 1250 0    60   ~ 0
 Incoming power filtering.\nIt is to not make input voltage \nvery low on powering up servos.
-Text Label 11350 2700 0    60   ~ 0
+Text Label 5700 7000 0    60   ~ 0
 pwr-en
 $Comp
@@
 Text Label 11150 9900 0    60   ~ 0
 pin_23
-Text Label 5700 7000 0    60   ~ 0
+Text Label 11350 2700 0    60   ~ 0
 pin_24
-Text Label 5450 8000 0    60   ~ 0
+Text Label 11350 6400 0    60   ~ 0
 pin_25
 $Comp
 L CONN_3 K5
 U 1 1 52B5BF19
-P 24400 1800
-F 0 "K5" V 24350 1800 50  0000 C CNN
-F 1 "CONN_3" V 24450 1800 40  0000 C CNN
-F 2 "" H 24400 1800 60  0000 C CNN
-F 3 "" H 24400 1800 60  0000 C CNN
-	1    24400 1800
+P 24400 2300
+F 0 "K5" V 24350 2300 50  0000 C CNN
+F 1 "CONN_3" V 24450 2300 40  0000 C CNN
+F 2 "" H 24400 2300 60  0000 C CNN
+F 3 "" H 24400 2300 60  0000 C CNN
+	1    24400 2300
 	1    0    0    -1
 $EndComp
@@
 L CONN_3 K6
 U 1 1 52B5E04A
-P 24400 2300
-F 0 "K6" V 24350 2300 50  0000 C CNN
-F 1 "CONN_3" V 24450 2300 40  0000 C CNN
-F 2 "" H 24400 2300 60  0000 C CNN
-F 3 "" H 24400 2300 60  0000 C CNN
-	1    24400 2300
+P 24400 2800
+F 0 "K6" V 24350 2800 50  0000 C CNN
+F 1 "CONN_3" V 24450 2800 40  0000 C CNN
+F 2 "" H 24400 2800 60  0000 C CNN
+F 3 "" H 24400 2800 60  0000 C CNN
+	1    24400 2800
 	1    0    0    -1
 $EndComp
@@
 L CONN_3 K7
 U 1 1 52B5E05C
-P 24400 2800
-F 0 "K7" V 24350 2800 50  0000 C CNN
-F 1 "CONN_3" V 24450 2800 40  0000 C CNN
-F 2 "" H 24400 2800 60  0000 C CNN
-F 3 "" H 24400 2800 60  0000 C CNN
-	1    24400 2800
+P 24400 3300
+F 0 "K7" V 24350 3300 50  0000 C CNN
+F 1 "CONN_3" V 24450 3300 40  0000 C CNN
+F 2 "" H 24400 3300 60  0000 C CNN
+F 3 "" H 24400 3300 60  0000 C CNN
+	1    24400 3300
 	1    0    0    -1
 $EndComp
@@
 L CONN_3 K8
 U 1 1 52B5E06E
-P 24400 3300
-F 0 "K8" V 24350 3300 50  0000 C CNN
-F 1 "CONN_3" V 24450 3300 40  0000 C CNN
-F 2 "" H 24400 3300 60  0000 C CNN
-F 3 "" H 24400 3300 60  0000 C CNN
-	1    24400 3300
+P 24400 3800
+F 0 "K8" V 24350 3800 50  0000 C CNN
+F 1 "CONN_3" V 24450 3800 40  0000 C CNN
+F 2 "" H 24400 3800 60  0000 C CNN
+F 3 "" H 24400 3800 60  0000 C CNN
+	1    24400 3800
 	1    0    0    -1
 $EndComp
@@
 L CONN_3 K9
 U 1 1 52B5E080
-P 24400 3800
-F 0 "K9" V 24350 3800 50  0000 C CNN
-F 1 "CONN_3" V 24450 3800 40  0000 C CNN
-F 2 "" H 24400 3800 60  0000 C CNN
-F 3 "" H 24400 3800 60  0000 C CNN
-	1    24400 3800
+P 24400 4300
+F 0 "K9" V 24350 4300 50  0000 C CNN
+F 1 "CONN_3" V 24450 4300 40  0000 C CNN
+F 2 "" H 24400 4300 60  0000 C CNN
+F 3 "" H 24400 4300 60  0000 C CNN
+	1    24400 4300
 	1    0    0    -1
 $EndComp
@@
 L CONN_3 K10
 U 1 1 52B5E092
-P 24400 4300
-F 0 "K10" V 24350 4300 50  0000 C CNN
-F 1 "CONN_3" V 24450 4300 40  0000 C CNN
-F 2 "" H 24400 4300 60  0000 C CNN
-F 3 "" H 24400 4300 60  0000 C CNN
-	1    24400 4300
+P 24400 4800
+F 0 "K10" V 24350 4800 50  0000 C CNN
+F 1 "CONN_3" V 24450 4800 40  0000 C CNN
+F 2 "" H 24400 4800 60  0000 C CNN
+F 3 "" H 24400 4800 60  0000 C CNN
+	1    24400 4800
 	1    0    0    -1
 $EndComp
@@
 L CONN_3 K11
 U 1 1 52B5E0A4
-P 24400 4800
-F 0 "K11" V 24350 4800 50  0000 C CNN
-F 1 "CONN_3" V 24450 4800 40  0000 C CNN
-F 2 "" H 24400 4800 60  0000 C CNN
-F 3 "" H 24400 4800 60  0000 C CNN
-	1    24400 4800
+P 24400 5300
+F 0 "K11" V 24350 5300 50  0000 C CNN
+F 1 "CONN_3" V 24450 5300 40  0000 C CNN
+F 2 "" H 24400 5300 60  0000 C CNN
+F 3 "" H 24400 5300 60  0000 C CNN
+	1    24400 5300
 	1    0    0    -1
 $EndComp
@@
 L CONN_3 K12
 U 1 1 52B5E0B6
-P 24400 5300
-F 0 "K12" V 24350 5300 50  0000 C CNN
-F 1 "CONN_3" V 24450 5300 40  0000 C CNN
-F 2 "" H 24400 5300 60  0000 C CNN
-F 3 "" H 24400 5300 60  0000 C CNN
-	1    24400 5300
+P 24400 8300
+F 0 "K12" V 24350 8300 50  0000 C CNN
+F 1 "CONN_3" V 24450 8300 40  0000 C CNN
+F 2 "" H 24400 8300 60  0000 C CNN
+F 3 "" H 24400 8300 60  0000 C CNN
+	1    24400 8300
 	1    0    0    -1
 $EndComp
@@
 	1    0    0    -1
 $EndComp
-Text Label 11350 6400 0    60   ~ 0
-pin_25
+Text Label 5450 8000 0    60   ~ 0
+pin_28
 Text Label 11350 6600 0    60   ~ 0
 pin_26
@@
 L CONN_3 K18
 U 1 1 52B5E79D
-P 24400 8300
-F 0 "K18" V 24350 8300 50  0000 C CNN
-F 1 "CONN_3" V 24450 8300 40  0000 C CNN
-F 2 "" H 24400 8300 60  0000 C CNN
-F 3 "" H 24400 8300 60  0000 C CNN
-	1    24400 8300
+P 24400 8800
+F 0 "K18" V 24350 8800 50  0000 C CNN
+F 1 "CONN_3" V 24450 8800 40  0000 C CNN
+F 2 "" H 24400 8800 60  0000 C CNN
+F 3 "" H 24400 8800 60  0000 C CNN
+	1    24400 8800
 	1    0    0    -1
 $EndComp
@@
 L CONN_3 K19
 U 1 1 52B5E7AF
-P 24400 8800
-F 0 "K19" V 24350 8800 50  0000 C CNN
-F 1 "CONN_3" V 24450 8800 40  0000 C CNN
-F 2 "" H 24400 8800 60  0000 C CNN
-F 3 "" H 24400 8800 60  0000 C CNN
-	1    24400 8800
+P 24400 1800
+F 0 "K19" V 24350 1800 50  0000 C CNN
+F 1 "CONN_3" V 24450 1800 40  0000 C CNN
+F 2 "" H 24400 1800 60  0000 C CNN
+F 3 "" H 24400 1800 60  0000 C CNN
+	1    24400 1800
 	1    0    0    -1
 $EndComp
@@
 	15300 2200 15300 2100
 Wire Wire Line
-	15500 2200 15500 2100
+	15500 2100 15500 2200
 Wire Wire Line
 	23500 1700 24050 1700
@@
 Wire Wire Line
 	10800 4400 11650 4400
+$Comp
+L CONN_3 K33
+U 1 1 52B74495
+P 24400 15800
+F 0 "K33" V 24350 15800 50  0000 C CNN
+F 1 "CONN_3" V 24450 15800 40  0000 C CNN
+F 2 "" H 24400 15800 60  0000 C CNN
+F 3 "" H 24400 15800 60  0000 C CNN
+	1    24400 15800
+	1    0    0    -1
+$EndComp
+Text Label 23550 15800 0    60   ~ 0
+pwr-servo
+Text Label 23550 15700 0    60   ~ 0
+pin_28
+$Comp
+L GND #PWR060
+U 1 1 52B7449D
+P 23950 16000
+F 0 "#PWR060" H 23950 16000 30  0001 C CNN
+F 1 "GND" H 23950 15930 30  0001 C CNN
+F 2 "" H 23950 16000 60  0000 C CNN
+F 3 "" H 23950 16000 60  0000 C CNN
+	1    23950 16000
+	1    0    0    -1
+$EndComp
+Wire Wire Line
+	24050 15900 23950 15900
+Wire Wire Line
+	23950 15900 23950 16000
+Wire Wire Line
+	24050 15800 23500 15800
+Wire Wire Line
+	23500 15700 24050 15700
 $EndSCHEMATC
